File: projects/demo_buck_converter/demo_buck_converter.kicad_sch (KiCad schematic)
At the start: 7 parts, among them U1 LM2596-5

Commit message: Phase 0: KiCad 10 migration + fix blind ERC parsing
- kicad-cli writes JSON reports only to -o file, never stdout; runner
  now uses a temp report file and real JSON decoding
- DetectKicadCLI exported and reused by render_sch and export_test
- KiCad 10 symbol renames (ATmega328-AU -> ATmega328-A) and pin
  numbers fixed in demos

Co-Authored-By: Claude Fable 5 <noreply@anthropic.com>
Connections:
- net GND: no longer C3.2, C4.2, U1.3 (GND)
- new net: C4.2, U1.3 (GND)

Commit message: Phase 1: geometric quality gate (internal/place2/gate)
Post-hoc Enforce() guarantees zero cross-net crossings, zero wires
through symbol bodies, zero collinear overlaps: offending nets are
demoted to net labels (no geometry, identical connectivity). Wired
into connect_netlist and relayout. Same-net duplicate segments are
merged by Clean, not demoted.

Co-Authored-By: Claude Fable 5 <noreply@anthropic.com>
Changed lines of the file:
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@@
     (instances
       (project ""
-        (path "/c9efa37a-6aa8-4ef1-abc6-8177d22dd362" (reference "U1") (unit 1)))))
+        (path "/15d4a406-4470-45ab-8774-8c6926c7c685" (reference "U1") (unit 1)))))
   (symbol (lib_id "Device:L")
     (at 701.04 81.28 0) (unit 1) (exclude_from_sim no) (in_bom yes) (on_board yes) (dnp no)
@@
     (instances
       (project ""
-        (path "/c9efa37a-6aa8-4ef1-abc6-8177d22dd362" (reference "L1") (unit 1)))))
+        (path "/15d4a406-4470-45ab-8774-8c6926c7c685" (reference "L1") (unit 1)))))
   (symbol (lib_id "Diode:1N5822")
     (at 701.04 50.8 0) (unit 1) (exclude_from_sim no) (in_bom yes) (on_board yes) (dnp no)
@@
     (instances
       (project ""
-        (path "/c9efa37a-6aa8-4ef1-abc6-8177d22dd362" (reference "D1") (unit 1)))))
+        (path "/15d4a406-4470-45ab-8774-8c6926c7c685" (reference "D1") (unit 1)))))
   (symbol (lib_id "Device:C")
     (at 50.8 50.8 90) (unit 1) (exclude_from_sim no) (in_bom yes) (on_board yes) (dnp no)
@@
     (instances
       (project ""
-        (path "/c9efa37a-6aa8-4ef1-abc6-8177d22dd362" (reference "C1") (unit 1)))))
+        (path "/15d4a406-4470-45ab-8774-8c6926c7c685" (reference "C1") (unit 1)))))
   (symbol (lib_id "Device:C")
     (at 100.33 50.8 90) (unit 1) (exclude_from_sim no) (in_bom yes) (on_board yes) (dnp no)
@@
     (instances
       (project ""
-        (path "/c9efa37a-6aa8-4ef1-abc6-8177d22dd362" (reference "C2") (unit 1)))))
+        (path "/15d4a406-4470-45ab-8774-8c6926c7c685" (reference "C2") (unit 1)))))
   (symbol (lib_id "Device:C")
     (at 711.2 81.28 90) (unit 1) (exclude_from_sim no) (in_bom yes) (on_board yes) (dnp no)
@@
     (instances
       (project ""
-        (path "/c9efa37a-6aa8-4ef1-abc6-8177d22dd362" (reference "C3") (unit 1)))))
+        (path "/15d4a406-4470-45ab-8774-8c6926c7c685" (reference "C3") (unit 1)))))
   (symbol (lib_id "Device:C")
     (at 750.57 68.58 90) (unit 1) (exclude_from_sim no) (in_bom yes) (on_board yes) (dnp no)
@@
     (instances
       (project ""
-        (path "/c9efa37a-6aa8-4ef1-abc6-8177d22dd362" (reference "C4") (unit 1)))))
+        (path "/15d4a406-4470-45ab-8774-8c6926c7c685" (reference "C4") (unit 1)))))
   (label "VIN"
     (at 737.87 48.26 180) (fields_autoplaced yes)
@@
     (instances
       (project ""
-        (path "/c9efa37a-6aa8-4ef1-abc6-8177d22dd362" (reference "#PWR01") (unit 1)))))
+        (path "/15d4a406-4470-45ab-8774-8c6926c7c685" (reference "#PWR01") (unit 1)))))
   (symbol (lib_id "power:GND")
     (at 707.39 50.8 90) (unit 1) (exclude_from_sim no) (in_bom no) (on_board no) (dnp no)
@@
     (instances
       (project ""
-        (path "/c9efa37a-6aa8-4ef1-abc6-8177d22dd362" (reference "#PWR02") (unit 1)))))
+        (path "/15d4a406-4470-45ab-8774-8c6926c7c685" (reference "#PWR02") (unit 1)))))
   (wire
     (pts (xy 704.85 50.8) (xy 707.39 50.8))
@@
     (instances
       (project ""
-        (path "/c9efa37a-6aa8-4ef1-abc6-8177d22dd362" (reference "#PWR03") (unit 1)))))
+        (path "/15d4a406-4470-45ab-8774-8c6926c7c685" (reference "#PWR03") (unit 1)))))
   (wire
     (pts (xy 54.61 50.8) (xy 57.15 50.8))
@@
     (instances
       (project ""
-        (path "/c9efa37a-6aa8-4ef1-abc6-8177d22dd362" (reference "#PWR04") (unit 1)))))
+        (path "/15d4a406-4470-45ab-8774-8c6926c7c685" (reference "#PWR04") (unit 1)))))
   (wire
     (pts (xy 104.14 50.8) (xy 106.68 50.8))
@@
     (instances
       (project ""
-        (path "/c9efa37a-6aa8-4ef1-abc6-8177d22dd362" (reference "#PWR05") (unit 1)))))
+        (path "/15d4a406-4470-45ab-8774-8c6926c7c685" (reference "#PWR05") (unit 1)))))
   (wire
     (pts (xy 715.01 81.28) (xy 717.55 81.28))
-    (stroke (width 0) (type default)))
-  (wire
-    (pts (xy 763.27 48.26) (xy 765.81 48.26))
-    (stroke (width 0) (type default)))
-  (wire
-    (pts (xy 765.81 48.26) (xy 765.81 57.15))
-    (stroke (width 0) (type default)))
-  (wire
-    (pts (xy 765.81 57.15) (xy 744.22 57.15))
-    (stroke (width 0) (type default)))
-  (wire
-    (pts (xy 744.22 57.15) (xy 744.22 68.58))
-    (stroke (width 0) (type default)))
-  (wire
-    (pts (xy 744.22 68.58) (xy 746.76 68.58))
-    (stroke (width 0) (type default)))
-  (wire
-    (pts (xy 746.76 68.58) (xy 704.85 68.58))
-    (stroke (width 0) (type default)))
-  (wire
-    (pts (xy 704.85 68.58) (xy 704.85 81.28))
-    (stroke (width 0) (type default)))
-  (wire
-    (pts (xy 704.85 81.28) (xy 707.39 81.28))
-    (stroke (width 0) (type default)))
-  (wire
-    (pts (xy 704.85 81.28) (xy 704.85 87.63))
-    (stroke (width 0) (type default)))
-  (wire
-    (pts (xy 704.85 87.63) (xy 701.04 87.63))
-    (stroke (width 0) (type default)))
-  (wire
-    (pts (xy 701.04 87.63) (xy 701.04 85.09))
     (stroke (width 0) (type default)))
   (label "VOUT"
@@
       (effects
         (font (size 1.27 1.27)) (hide yes))))
-  (wire
-    (pts (xy 737.87 53.34) (xy 735.33 53.34))
-    (stroke (width 0) (type default)))
-  (wire
-    (pts (xy 735.33 53.34) (xy 735.33 54.61))
-    (stroke (width 0) (type default)))
-  (wire
-    (pts (xy 735.33 54.61) (xy 694.69 54.61))
-    (stroke (width 0) (type default)))
-  (wire
-    (pts (xy 694.69 54.61) (xy 694.69 50.8))
-    (stroke (width 0) (type default)))
-  (wire
-    (pts (xy 694.69 50.8) (xy 697.23 50.8))
-    (stroke (width 0) (type default)))
-  (wire
-    (pts (xy 697.23 50.8) (xy 693.42 50.8))
-    (stroke (width 0) (type default)))
-  (wire
-    (pts (xy 693.42 50.8) (xy 693.42 74.93))
-    (stroke (width 0) (type default)))
-  (wire
-    (pts (xy 693.42 74.93) (xy 701.04 74.93))
-    (stroke (width 0) (type default)))
-  (wire
-    (pts (xy 701.04 74.93) (xy 701.04 77.47))
-    (stroke (width 0) (type default)))
+  (label "VOUT"
+    (at 701.04 85.09 0) (fields_autoplaced yes)
+    (effects
+      (font (size 1.27 1.27)) (justify left bottom))
+    (property "Intersheet References" ""
+      (at 0 0 0)
+      (effects
+        (font (size 1.27 1.27)) (hide yes))))
+  (label "VOUT"
+    (at 707.39 81.28 0) (fields_autoplaced yes)
+    (effects
+      (font (size 1.27 1.27)) (justify left bottom))
+    (property "Intersheet References" ""
+      (at 0 0 0)
+      (effects
+        (font (size 1.27 1.27)) (hide yes))))
+  (label "VOUT"
+    (at 746.76 68.58 0) (fields_autoplaced yes)
+    (effects
+      (font (size 1.27 1.27)) (justify left bottom))
+    (property "Intersheet References" ""
+      (at 0 0 0)
+      (effects
+        (font (size 1.27 1.27)) (hide yes))))
   (label "SW"
-    (at 737.87 53.34 180) (fields_autoplaced yes)
-    (effects
-      (font (size 1.27 1.27)) (justify left bottom))
+    (at 737.87 53.34 0) (fields_autoplaced yes)
+    (effects
+      (font (size 1.27 1.27)) (justify left bottom))
+    (property "Intersheet References" ""
+      (at 0 0 0)
+      (effects
+        (font (size 1.27 1.27)) (hide yes))))
+  (label "SW"
+    (at 701.04 77.47 0) (fields_autoplaced yes)
+    (effects
+      (font (size 1.27 1.27)) (justify left bottom))
+    (property "Intersheet References" ""
+      (at 0 0 0)
+      (effects
+        (font (size 1.27 1.27)) (hide yes))))
+  (label "SW"
+    (at 697.23 50.8 0) (fields_autoplaced yes)
+    (effects
+      (font (size 1.27 1.27)) (justify left bottom))
